Commit message: changed urdf.xacro palm rpy

File: urdf/ur5e.xacro (robot description, xacro)
@@ -53,10 +53,9 @@
   </joint>
   <!-- Describe the location of the palm -->
-  FIX THIS AHHHHHHHHH
   <joint name="hand_palm" type="fixed">
     <parent link="tool0" />
     <child link="palm" />
 <!--        <origin xyz="0 0 0.13" rpy="0 0 0.2618 " />      &lt;!&ndash; Add in Z the hand's thickness (approx 13cm) &ndash;&gt;-->
-    <origin xyz="0 0 .165" rpy="0 0 -1.57 " />      <!-- Add in Z the hand's thickness (approx 13cm) -->
+    <origin xyz="0 0 .165" rpy="0 0 -1.20 " />      <!-- Add in Z the hand's thickness (approx 13cm) -->
   </joint>
   <!-- <joint name = "apple_proxy" type = "fixed">

Commit message: shifted apple location, may need more fine tuning

File: urdf/ur5e.xacro (robot description, xacro)
@@ -76,5 +76,5 @@
     <child link = "apple" />
     <!-- <origin xyz = "-0.04 -0.03 -2.08" rpy="0 0.0 0.0" /> -->
-    <origin xyz = "-.95 -.12 .5225" rpy="0 0 0" />
+    <origin xyz = "-.95 -.14 .5225" rpy="0 0 0" />
   </joint>
 </robot>

Commit message: adjusted workspace and angles

File: urdf/ur5e.xacro (robot description, xacro)
@@ -57,5 +57,5 @@
     <child link="palm" />
 <!--        <origin xyz="0 0 0.13" rpy="0 0 0.2618 " />      &lt;!&ndash; Add in Z the hand's thickness (approx 13cm) &ndash;&gt;-->
-    <origin xyz="0 0 .165" rpy="0 0 -1.20 " />      <!-- Add in Z the hand's thickness (approx 13cm) -->
+    <origin xyz="0 0 .165" rpy="0 0 -1.36 " />      <!-- Add in Z the hand's thickness (approx 13cm) -1.20-->
   </joint>
   <!-- <joint name = "apple_proxy" type = "fixed">
@@ -76,5 +76,5 @@
     <child link = "apple" />
     <!-- <origin xyz = "-0.04 -0.03 -2.08" rpy="0 0.0 0.0" /> -->
-    <origin xyz = "-.95 -.14 .5225" rpy="0 0 0" />
+    <origin xyz = "-1.02 -.09 .505" rpy="0 0 0" />
   </joint>
 </robot>

Commit message: updated apple start pos

File: urdf/ur5e.xacro (robot description, xacro)
@@ -75,6 +75,6 @@
     <parent link = "base_link" />
     <child link = "apple" />
-    <!-- <origin xyz = "-0.04 -0.03 -2.08" rpy="0 0.0 0.0" /> -->
-    <origin xyz = "-1.02 -.09 .505" rpy="0 0 0" />
+    <!-- <origin xyz = "-1.02 -.09 .505" rpy="0 0 0" /> -->
+    <origin xyz = "-1.075 -.095 .505" rpy = "0 0 0" />
   </joint>
 </robot>

Commit message: apple pos is updated... better angles now!

File: urdf/ur5e.xacro (robot description, xacro)
@@ -66,5 +66,5 @@
   <!--</joint> -->
   <joint name = "proxy_stem" type="fixed">
-    <parent link = "base_link" />
+    <parent link = "base_link" /> -m
     <child link = "apple_stem" />
     <!-- <origin xyz = "0.16 0.45 2.42" rpy="0 3.1416 0.0" /> -->
@@ -76,5 +76,5 @@
     <child link = "apple" />
     <!-- <origin xyz = "-1.02 -.09 .505" rpy="0 0 0" /> -->
-    <origin xyz = "-1.075 -.095 .505" rpy = "0 0 0" />
+    <origin xyz = "-1.075 -.095 .505" rpy = "0 0 0" /> <!--x was 1.055, may have shifted in the wrong direction-->
   </joint>
 </robot>
